File: _autosave-adin1110-featherwing.kicad_sch (KiCad schematic)
At the start: 58 parts, among them J1 4039_Header_Male_Vert_16pin_0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, J2 4040_Header_Male_Vert_12pin_0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, J3 4060_TerminalBlock_NoScrew, SW2 RST, T1 4057_Super_Tiny_Signal_Transf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, U1 4052_ADIN1110, U2 4058_TVS_2CH_Super_Speed, U3 LED0, U4 LED1, U5 LINK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

Commit message: as ordered for revA
Parts:
- TP2, TP3, TP4: footprint Shulltronics_Generics:TestPoint_Pad_D2.0mm -> Connector_Pin:Pin_D0.7mm_L6.5mm_W1.8mm_FlatFork
Changed lines of the file:
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@@
       (effects (font (size 1.27 1.27)) hide)
     )
-    (property "Footprint" "Shulltronics_Generics:TestPoint_Pad_D2.0mm" (at 249.555 111.76 0)
+    (property "Footprint" "Connector_Pin:Pin_D0.7mm_L6.5mm_W1.8mm_FlatFork" (at 249.555 111.76 0)
       (effects (font (size 1.27 1.27)) hide)
     )
@@
       (effects (font (size 1.27 1.27)) hide)
     )
-    (property "Footprint" "Shulltronics_Generics:TestPoint_Pad_D2.0mm" (at 222.25 111.76 0)
+    (property "Footprint" "Connector_Pin:Pin_D0.7mm_L6.5mm_W1.8mm_FlatFork" (at 222.25 111.76 0)
       (effects (font (size 1.27 1.27)) hide)
     )
@@
       (effects (font (size 1.27 1.27)) hide)
     )
-    (property "Footprint" "Shulltronics_Generics:TestPoint_Pad_D2.0mm" (at 193.675 111.76 0)
-      (effects (font (size 1.27 1.27)) hide)
-    )
+    (property "Footprint" "Connector_Pin:Pin_D0.7mm_L6.5mm_W1.8mm_FlatFork" (at 193.675 111.76 0)
+      (effects (font (size 1.27 1.27)) hide)
+    )
