File: adin1110-featherwing.kicad_sch (KiCad schematic)
At the start: 58 parts, among them J1 4039_Header_Male_Vert_16pin_0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, J2 4040_Header_Male_Vert_12pin_0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, J3 4060_TerminalBlock_NoScrew, SW2 RST, T1 4057_Super_Tiny_Signal_Transf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, U1 4052_ADIN1110, U2 4058_TVS_2CH_Super_Speed, U3 LED0, U4 LED1, U5 LINK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

Commit message: more rev 2 notes
Other:
- note added: "REV Double check footprint for pulse transformer.. it seems slightly off"
- note added: "REV LINK_ST LED has different polarity than the others!"
- note added: "REV TODO: Test all LED circuits and determine best resistance value."
- note added: "REV make sure 1->6 and 2->5 are connected with copper. Should probably alter footprint and symbol to achieve this."
- note added: "REV use smaller three pin screw terminal"
Changed lines of the file:
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@@
     (effects (font (size 1.27 1.27)) (justify left bottom))
+  )
+  (text "REV\nmake sure 1->6 and 2->5 are connected with copper.\nShould probably alter footprint and symbol to achieve this."
+    (at 171.45 19.05 0)
+    (effects (font (size 1.27 1.27) (color 255 0 0 1)) (justify left bottom))
   )
   (text "Feather Headers" (at 42.545 144.78 0)
     (effects (font (size 2.54 2.54) bold italic) (justify left bottom))
   )
+  (text "REV\nTODO: Test all LED circuits and\ndetermine best resistance value."
+    (at 190.5 91.44 0)
+    (effects (font (size 1.27 1.27) (color 255 0 0 1)) (justify left bottom))
+  )
+  (text "REV\nuse smaller three pin screw terminal" (at 247.65 30.48 0)
+    (effects (font (size 1.27 1.27) (color 255 0 0 1)) (justify left bottom))
+  )
+  (text "REV\nDouble check footprint for pulse transformer..\nit seems slightly off"
+    (at 203.2 78.74 0)
+    (effects (font (size 1.27 1.27) (color 255 0 0 1)) (justify left bottom))
+  )
+  (text "REV\nLINK_ST LED has different polarity than the others!"
+    (at 231.14 95.25 0)
+    (effects (font (size 1.27 1.27) (color 255 0 0 1)) (justify left bottom))
+  )
   (text "D3, D4, D5 (short header, pins 9, 8, 7)\nare hardwired by Particle Ethernet FW\nPin7 also used for CS by Adafruit Ethernet FW"
